Commit message: Add files via upload

File: urdf/si_amr.urdf (robot description, URDF)
Before this commit: robot si_amr, 10 links, 9 joints
Links:
- added link camera_front_view_link, mass 0.001
Joints:
- added joint camera_front_view_joint: type fixed, parent camera_front_link, child camera_front_view_link, origin xyz=0.0 0.0 0.0 rpy=-1.5708 0.0 -1.5708
- joint camera_front_joint: axis 0 0 0 -> 0 1 0
